Commit message: update

File: datasets/omnigibson-robot-assets/models/r1pro/urdf/r1pro_ik.urdf (robot description, URDF)
Before this commit: robot r1_pro_with_gripper, 36 links, 35 joints
Joints:
- joint torso_joint1: limit lower=-0.2 upper=0.2 effort=100 velocity=2.5 -> lower=-1 upper=1 effort=100 velocity=2.5
- joint torso_joint2: limit lower=-0.2 upper=0.2 effort=100 velocity=2.5 -> lower=-2.7925 upper=2.5307 effort=100 velocity=2.5
- joint torso_joint3: limit lower=-0.2 upper=0.2 effort=100 velocity=2.5 -> lower=-1 upper=1. effort=100 velocity=2.5
- joint torso_joint4: limit lower=-0.2 upper=0.2 effort=100 velocity=2.5 -> lower=-3.0543 upper=3.0543 effort=100 velocity=2.5
